Commit message: feat(arm): align control stack with fixed-yaw four-axis hardware

File: ros2_ws/src/robot_arm_description/urdf/robot_arm.urdf (robot description, URDF)
Before this commit: robot robot_arm, 52 links, 51 joints
Joints:
- joint arm_joint_1: axis 0.0 0.0 1.0 -> (none); type continuous -> fixed

File: ros2_ws/src/robot_arm_moveit_config/config/robot_arm.ros2_control.xacro (robot description, xacro)
@@ -8,11 +8,4 @@
                 <plugin>mock_components/GenericSystem</plugin>
             </hardware>
-            <joint name="arm_joint_1">
-                <command_interface name="position"/>
-                <state_interface name="position">
-                  <param name="initial_value">${initial_positions['arm_joint_1']}</param>
-                </state_interface>
-                <state_interface name="velocity"/>
-            </joint>
             <joint name="arm_joint_2">
                 <command_interface name="position"/>
